Commit message: add mrobot_tk1_home and edit the script before report to Mr. Zhou

File: mrobot_description/urdf/mrobot_body.urdf.xacro (robot description, xacro)
@@ -62,4 +62,94 @@
     </collision>
   </link>
+  <!--hjm add start -->
+  <link name="ultrasound_1">
+    <visual>
+       <geometry>
+         <box size="0.01 0.04 0.02"/>
+       </geometry>
+       <origin rpy="0 0 0" xyz="0 0 0"/>
+       <material name="red">
+         <color rgba="1 0 0 1"/>
+       </material>
+    </visual>
+  </link>
+  <joint
+    name="ultrasound_1_joint"
+    type="fixed">
+    <origin
+      xyz="0.0825 0.08 -0.0535"
+      rpy="0 0 0.5236" />
+    <parent
+      link="base_link" />
+    <child
+      link="ultrasound_1" />
+  </joint>
+  <link name="ultrasound_2">
+    <visual>
+       <geometry>
+         <box size="0.01 0.04 0.02"/>
+       </geometry>
+       <origin rpy="0 0 0" xyz="0 0 0"/>
+       <material name="red">
+         <color rgba="1 0 0 1"/>
+       </material>
+    </visual>
+  </link>
+  <joint
+    name="ultrasound_2_joint"
+    type="fixed">
+    <origin
+      xyz="0.112017059221718 0.03 -0.0535"
+      rpy="0 0 0.5236" />
+    <parent
+      link="base_link" />
+    <child
+      link="ultrasound_2" />
+  </joint>
+  <link name="ultrasound_3">
+    <visual>
+       <geometry>
+         <box size="0.01 0.04 0.02"/>
+       </geometry>
+       <origin rpy="0 0 0" xyz="0 0 0"/>
+       <material name="red">
+         <color rgba="1 0 0 1"/>
+       </material>
+    </visual>
+  </link>
+  <joint
+    name="ultrasound_3_joint"
+    type="fixed">
+    <origin
+      xyz="0.112017059221718 -0.03 -0.0535"
+      rpy="0 0 -0.5236" />
+    <parent
+      link="base_link" />
+    <child
+      link="ultrasound_3" />
+  </joint>
+  <link name="ultrasound_4">
+    <visual>
+       <geometry>
+         <box size="0.01 0.04 0.02"/>
+       </geometry>
+       <origin rpy="0 0 0" xyz="0 0 0"/>
+       <material name="red">
+         <color rgba="1 0 0 1"/>
+       </material>
+    </visual>
+  </link>
+  <joint
+    name="ultrasound_4_joint"
+    type="fixed">
+    <origin
+      xyz="0.0825 -0.08 -0.0535"
+      rpy="0 0 -0.5236" />
+    <parent
+      link="base_link" />
+    <child
+      link="ultrasound_4" />
+  </joint>
+  <!-- hjm add end -->
   <link
     name="XtionPro_Link">
